File: RP-006442-DD-2-RP2350B Minimal Board Kicad archive/RP2350_80QFN_minimal.kicad_pcb (KiCad board)
At the start: 2 copper layers, 92 x 98 mm, 94 parts, among them J1 USB_C_Receptacle_USB2.0_16P, J2 Conn_02x26_Odd_Even, J3 Conn_02x26_Odd_Even, J4 Conn_01x03, J5 USB_C_Receptacle_USB2.0_16P, SW1 SW_Push, SW2 SW_Push, SW3 SW_Push, SW4 SW_Push, U1 RP2350_80QFN, U2 NCP1117-3.3_SOT223, U3 W25Q128JVS, U4 DNF, U5 W25Q128JVS, U6 NCP1117-3.3_SOT223, U7 RP2350_60QFN, U8 HT16K33A-28SOP, U9 CC56-12EWA, Y1 ABM8-272-T3, Y2 ABM8-272-T3

Commit message: Update to pcb
Parts:
- moved SW2 2.44 mm to (108.3, 113.9)
- moved R4 2.44 mm to (105.7, 114.0)
- moved C37 0.88 mm to (152.5, 97.0)
Routing:
- net VBUS: track 16.7 -> 19.9 mm
- net /RUN: track 31.4 -> 32.5 mm
- net +3V3: track 79.0 -> 78.4 mm
Changed lines of the file:
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@@
 	(footprint "Resistor_SMD:R_0402_1005Metric"
 		(layer "F.Cu")
-		(at 108.1 113.7 -90)
+		(at 105.675 114 -90)
 		(descr "Resistor SMD 0402 (1005 Metric), square (rectangular) end terminal, IPC_7351 nominal, (Body size source: IPC-SM-782 page 72, https://www.pcb-3d.com/wordpress/wp-content/uploads/ipc-sm-782a_amendment_1_and_2.pdf), generated with kicad-footprint-generator")
 		(tags "resistor")
@@
 		(tags "capacitor")
 		(property "Reference" "C32"
-			(at 2.3 -0.1 0)
+			(at 2.4 -0.1 0)
 			(layer "F.SilkS")
 			(effects
@@
 	(footprint "Capacitor_SMD:C_0402_1005Metric"
 		(layer "F.Cu")
-		(at 153.28 97.4)
+		(at 152.5 97)
 		(descr "Capacitor SMD 0402 (1005 Metric), square (rectangular) end terminal, IPC_7351 nominal, (Body size source: IPC-SM-782 page 76, https://www.pcb-3d.com/wordpress/wp-content/uploads/ipc-sm-782a_amendment_1_and_2.pdf), generated with kicad-footprint-generator")
 		(tags "capacitor")
 		(property "Reference" "C37"
-			(at 2.3 0 0)
+			(at 2.42 0 0)
 			(layer "F.SilkS")
 			(effects
@@
 		(tags "capacitor")
 		(property "Reference" "C34"
-			(at 2.3 0.1 0)
+			(at 2.4 0.2 0)
 			(layer "F.SilkS")
 			(effects
@@
 	(footprint "Button_Switch_SMD:SW_Push_1P1T_NO_Vertical_Wuerth_434133025816"
 		(layer "F.Cu")
-		(at 110.725 113.6 90)
+		(at 108.3 113.9 90)
 		(descr "https://katalog.we-online.com/em/datasheet/434133025816.pdf")
 		(tags "tactile switch Wurth Wuerth")
@@
 			)
 		)
-		(pad "1" smd roundrect
+		(pad "1" smd rect
 			(at -3.15 -2.3 270)
 			(size 2 1.5)
 			(layers "F.Cu" "F.Mask" "F.Paste")
-			(roundrect_rratio 0.25)
 			(net 1 "GND")
 			(pinfunction "GND")
 			(pintype "power_in")
 		)
-		(pad "2" smd roundrect
+		(pad "2" smd rect
 			(at -3.15 0 270)
 			(size 2 1.5)
 			(layers "F.Cu" "F.Mask" "F.Paste")
-			(roundrect_rratio 0.25)
 			(net 5 "+3V3")
 			(pinfunction "VO")
 			(pintype "power_out")
 		)
-		(pad "2" smd roundrect
+		(pad "2" smd rect
 			(at 3.15 0 270)
 			(size 2 3.8)
 			(layers "F.Cu" "F.Mask" "F.Paste")
-			(roundrect_rratio 0.25)
 			(net 5 "+3V3")
 			(pinfunction "VO")
 			(pintype "power_out")
 		)
-		(pad "3" smd roundrect
+		(pad "3" smd rect
 			(at -3.15 2.3 270)
 			(size 2 1.5)
 			(layers "F.Cu" "F.Mask" "F.Paste")
-			(roundrect_rratio 0.25)
 			(net 2 "VBUS")
 			(pinfunction "VI")
@@
 	)
 	(segment
-		(start 108.1 114.18)
-		(end 108.1 115)
+		(start 105.675 114.48)
+		(end 105.675 115.3)
 		(width 0.15)
 		(layer "F.Cu")
@@
 	)
 	(via
-		(at 108.1 115)
+		(at 105.675 115.3)
 		(size 0.6)
 		(drill 0.25)
@@
 	)
 	(segment
+		(start 147.85 78.045)
+		(end 147.85 78.972)
+		(width 0.4)
+		(layer "F.Cu")
+		(net 2)
+	)
+	(segment
 		(start 144.00743 76.2)
 		(end 146.79257 76.2)
@@
 	)
 	(segment
+		(start 147.85 78.972)
+		(end 149.478 80.6)
+		(width 0.4)
+		(layer "F.Cu")
+		(net 2)
+	)
+	(segment
 		(start 102.45 77.25743)
 		(end 102.45 78.045)
@@
 	)
 	(segment
-		(start 149.86973 97.729)
-		(end 152.471 97.729)
-		(width 0.2)
-		(layer "F.Cu")
-		(net 5)
-	)
-	(segment
 		(start 145.23223 103.5665)
 		(end 145.23 103.56427)
@@
 	)
 	(segment
-		(start 152.471 97.729)
-		(end 152.8 97.4)
-		(width 0.2)
-		(layer "F.Cu")
-		(net 5)
-	)
-	(segment
 		(start 106.3 100.2)
 		(end 106.6 100.5)
@@
 	)
 	(segment
+		(start 151.4 97)
+		(end 152.02 97)
+		(width 0.15)
+		(layer "F.Cu")
+		(net 5)
+	)
+	(segment
 		(start 104.8965 100.2)
 		(end 103.8 100.2)
@@
 	)
 	(segment
+		(start 149.86973 97.729)
+		(end 150.671 97.729)
+		(width 0.15)
+		(layer "F.Cu")
+		(net 5)
+	)
+	(segment
 		(start 152.115623 100.4)
 		(end 153.02 100.4)
@@
 	)
 	(segment
+		(start 150.671 97.729)
+		(end 151.4 97)
+		(width 0.15)
+		(layer "F.Cu")
+		(net 5)
+	)
+	(segment
 		(start 100.6 94.2)
 		(end 100.6 95.1035)
@@
 	)
 	(segment
-		(start 111.8 115.675)
-		(end 112.465 115.675)
+		(start 101.8 106)
+		(end 104 108.2)
 		(width 0.15)
 		(layer "F.Cu")
@@
 	)
 	(segment
-		(start 101.8 106)
-		(end 104 108.2)
+		(start 109.375 109.475)
+		(end 108.1 108.2)
 		(width 0.15)
 		(layer "F.Cu")
@@
 	)
 	(segment
-		(start 111.8 111)
-		(end 111.8 111.55)
+		(start 109.375 111.85)
+		(end 109.375 109.475)
 		(width 0.15)
 		(layer "F.Cu")
@@
 	)
 	(segment
-		(start 111.8 115.675)
-		(end 111.8 111.55)
+		(start 112.765 115.975)
+		(end 121.59 124.8)
 		(width 0.15)
 		(layer "F.Cu")
@@
 	)
 	(segment
-		(start 101.8 104.8965)
-		(end 101.8 106)
+		(start 109.375 115.975)
+		(end 109.375 111.85)
 		(width 0.15)
 		(layer "F.Cu")
@@
 	)
 	(segment
-		(start 109 108.2)
-		(end 111.8 111)
+		(start 109.375 115.975)
+		(end 112.765 115.975)
 		(width 0.15)
 		(layer "F.Cu")
@@
 	)
 	(segment
-		(start 112.465 115.675)
-		(end 121.59 124.8)
+		(start 101.8 104.8965)
+		(end 101.8 106)
 		(width 0.15)
 		(layer "F.Cu")
@@
 	(segment
 		(start 104 108.2)
-		(end 109 108.2)
+		(end 108.1 108.2)
 		(width 0.15)
 		(layer "F.Cu")
@@
 	)
 	(segment
+		(start 107.3 110.6)
+		(end 105.3 110.6)
+		(width 0.15)
+		(layer "F.Cu")
+		(net 36)
+	)
+	(segment
 		(start 101 106.3)
 		(end 101 104.8965)
@@
 	)
 	(segment
-		(start 108.2 109.9)
-		(end 104.6 109.9)
-		(width 0.15)
-		(layer "F.Cu")
-		(net 36)
-	)
-	(segment
-		(start 104.6 109.9)
+		(start 105.3 110.6)
 		(end 101 106.3)
 		(width 0.15)
@@
 	)
 	(via
-		(at 108.2 109.9)
+		(at 107.3 110.6)
 		(size 0.6)
 		(drill 0.35)
@@
 	(segment
 		(start 126.164 110.636)
-		(end 108.936 110.636)
+		(end 130.1 106.7)
 		(width 0.15)
 		(layer "B.Cu")
@@
 	)
 	(segment
-		(start 108.936 110.636)
-		(end 108.2 109.9)
+		(start 107.336 110.636)
+		(end 126.164 110.636)
 		(width 0.15)
 		(layer "B.Cu")
@@
 	)
 	(segment
-		(start 130.1 106.7)
-		(end 126.164 110.636)
+		(start 107.3 110.6)
+		(end 107.336 110.636)
 		(width 0.15)
 		(layer "B.Cu")
@@
 	)
 	(segment
-		(start 130.1 103.5)
-		(end 130.1 106.7)
+		(start 130.1 106.7)
+		(end 130.1 103.5)
 		(width 0.15)
 		(layer "B.Cu")
@@
 	)
 	(segment
-		(start 109.705 113.22)
-		(end 109.725 113.2)
+		(start 105.675 113.52)
+		(end 105.695 113.5)
 		(width 0.15)
 		(layer "F.Cu")
@@
 	)
 	(segment
-		(start 109.725 111.525)
-		(end 109.725 113.2)
+		(start 105.695 113.5)
+		(end 107.26 113.5)
 		(width 0.15)
 		(layer "F.Cu")
@@
 	)
 	(segment
-		(start 108.1 113.22)
-		(end 109.705 113.22)
+		(start 107.26 113.5)
+		(end 107.28 113.52)
 		(width 0.15)
 		(layer "F.Cu")
@@
 	)
 	(segment
-		(start 109.725 113.2)
-		(end 109.725 115.675)
+		(start 107.3 111.825)
+		(end 107.3 113.5)
+		(width 0.15)
+		(layer "F.Cu")
+		(net 65)
+	)
+	(segment
+		(start 107.3 113.5)
+		(end 107.3 115.975)
 		(width 0.15)
 		(layer "F.Cu")
@@
 	)
 	(zone
+		(net 5)
+		(net_name "+3V3")
+		(layer "F.Cu")
+		(hatch edge 0.5)
+		(priority 12)
+		(connect_pads
+			(clearance 0.2)
+		)
+		(min_thickness 0.15)
+		(filled_areas_thickness no)
+		(fill yes
+			(thermal_gap 0.5)
+			(thermal_bridge_width 0.5)
+		)
+		(polygon
+			(pts
+				(xy 127 70.5) (xy 127.1 115.4) (xy 165.5 115.4) (xy 165.5 70.5)
+			)
+		)
+	)
+	(zone
+		(net 0)
+		(net_name "")
+		(layer "F.Cu")
+		(hatch edge 0.5)
+		(connect_pads
+			(clearance 0)
+		)
+		(min_thickness 0.25)
+		(filled_areas_thickness no)
+		(keepout
+			(tracks allowed)
+			(vias allowed)
+			(pads allowed)
+			(copperpour not_allowed)
+			(footprints allowed)
+		)
+		(placement
+			(enabled no)
+			(sheetname "")
+		)
+		(fill
+			(thermal_gap 0.5)
+			(thermal_bridge_width 0.5)
+		)
+		(polygon
+			(pts
+				(xy 149.3 98.1) (xy 149.3 97.6) (xy 149.4 97.5) (xy 150.6 97.5) (xy 151.4 96.7) (xy 151.8 96.7)
+				(xy 151.8 97.2) (xy 151.4 97.2) (xy 150.5 98.1)
+			)
+		)
+	)
+	(zone
 		(net 0)
 		(net_name "")
@@
 		(polygon
 			(pts
+				(xy 143.6 96.5) (xy 142.8 96.5) (xy 142.8 103.1) (xy 143.528571 103.1) (xy 143.6 102.9)
+			)
+		)
+	)
+	(zone
+		(net 0)
+		(net_name "")
+		(layer "F.Cu")
+		(hatch edge 0.5)
+		(connect_pads
+			(clearance 0)
+		)
+		(min_thickness 0.25)
+		(filled_areas_thickness no)
+		(keepout
+			(tracks allowed)
+			(vias allowed)
+			(pads allowed)
+			(copperpour not_allowed)
+			(footprints allowed)
+		)
+		(placement
+			(enabled no)
+			(sheetname "")
+		)
+		(fill
+			(thermal_gap 0.5)
+			(thermal_bridge_width 0.5)
+		)
+		(polygon
+			(pts
 				(xy 96 104.2) (xy 95.9 104.3) (xy 95.9 105) (xy 104 105) (xy 104 104.4) (xy 103.8 104.2)
 			)
@@
 		(layer "F.Cu")
 		(hatch edge 0.5)
-		(priority 11)
+		(priority 15)
 		(connect_pads
 			(clearance 0.15)
@@
 		(polygon
 			(pts
-				(xy 148.5 79.75) (xy 148.5 85.5) (xy 153 85.5) (xy 153 82) (xy 155 82) (xy 155 78.75) (xy 151 78.75)
-				(xy 151 79.75)
+				(xy 146.6 79.75) (xy 146.6 85.5) (xy 152.3 85.5) (xy 152.3 82) (xy 155 82) (xy 155 77.65) (xy 150.2 77.65)
+				(xy 150.2 79.75)
 			)
 		)

Commit message: Update to pcb
Parts:
- moved R23 0.10 mm to (147.4, 80.3)
Routing:
- net GND: track 65.8 -> 66.6 mm
Changed lines of the file:
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@@
 	(footprint "Resistor_SMD:R_0402_1005Metric"
 		(layer "F.Cu")
-		(at 147.3 80.3 90)
+		(at 147.4 80.3 90)
 		(descr "Resistor SMD 0402 (1005 Metric), square (rectangular) end terminal, IPC_7351 nominal, (Body size source: IPC-SM-782 page 72, https://www.pcb-3d.com/wordpress/wp-content/uploads/ipc-sm-782a_amendment_1_and_2.pdf), generated with kicad-footprint-generator")
 		(tags "resistor")
@@
 	)
 	(segment
+		(start 144.1 92.32)
+		(end 144.1 91.5)
+		(width 0.15)
+		(layer "F.Cu")
+		(net 1)
+	)
+	(segment
 		(start 108.8875 78.75)
 		(end 109.8875 79.75)
@@
 	)
 	(segment
-		(start 147.3 80.81)
-		(end 147.3 81.6)
+		(start 147.4 80.81)
+		(end 147.4 81.6)
 		(width 0.2)
 		(layer "F.Cu")
@@
 	)
 	(via
-		(at 147.3 81.6)
+		(at 147.4 81.6)
 		(size 0.6)
 		(drill 0.35)
@@
 	)
 	(zone
+		(net 0)
+		(net_name "")
+		(layer "F.Cu")
+		(hatch edge 0.508)
+		(connect_pads
+			(clearance 0)
+		)
+		(min_thickness 0.2)
+		(filled_areas_thickness no)
+		(keepout
+			(tracks allowed)
+			(vias allowed)
+			(pads allowed)
+			(copperpour not_allowed)
+			(footprints allowed)
+		)
+		(placement
+			(enabled no)
+			(sheetname "/")
+		)
+		(fill
+			(thermal_gap 0.3)
+			(thermal_bridge_width 0.3)
+		)
+		(polygon
+			(pts
+				(xy 143.7 88.2) (xy 144.5 88.2) (xy 144.5 91.2) (xy 143.7 91.2)
+			)
+		)
+	)
+	(zone
 		(net 6)
 		(net_name "+1V1")
@@
 		(layer "F.Cu")
 		(hatch edge 0.508)
-		(priority 10)
+		(priority 20)
 		(connect_pads
 			(clearance 0.2)
@@
 		(net_name "")
 		(layer "F.Cu")
+		(hatch edge 0.508)
+		(connect_pads
+			(clearance 0)
+		)
+		(min_thickness 0.15)
+		(filled_areas_thickness no)
+		(keepout
+			(tracks allowed)
+			(vias allowed)
+			(pads allowed)
+			(copperpour not_allowed)
+			(footprints allowed)
+		)
+		(placement
+			(enabled no)
+			(sheetname "")
+		)
+		(fill
+			(thermal_gap 0.3)
+			(thermal_bridge_width 0.3)
+		)
+		(polygon
+			(pts
+				(xy 133.5 85.2) (xy 133.5 90) (xy 138.6 90) (xy 143.3 94.7) (xy 145.1 94.7) (xy 145.1 92.083333)
+				(xy 141.4 89) (xy 141.4 85.2)
+			)
+		)
+	)
+	(zone
+		(net 0)
+		(net_name "")
+		(layer "F.Cu")
 		(hatch edge 0.5)
 		(connect_pads
@@
 			)
 		)
+	)
+	(zone
+		(net 0)
+		(net_name "")
+		(layer "F.Cu")
+		(hatch edge 0.508)
+		(connect_pads
+			(clearance 0)
+		)
+		(min_thickness 0.15)
+		(filled_areas_thickness no)
+		(keepout
+			(tracks allowed)
+			(vias allowed)
+			(pads allowed)
+			(copperpour not_allowed)
+			(footprints allowed)
+		)
+		(placement
+			(enabled no)
+			(sheetname "")
+		)
+		(fill
+			(thermal_gap 0.3)
+			(thermal_bridge_width 0.3)
+		)
+		(polygon
+			(pts
+				(xy 144.8125 79.15) (xy 146.9 79.15) (xy 146.9 90.2) (xy 146.9 88.4) (xy 146.9 91.4) (xy 144.1 91.4)
+				(xy 144.1 78.9)
+			)
+		)

Commit message: Update to pcb
Routing:
- net /RUN: track 32.5 -> 16.6 mm
Changed lines of the file:
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@@
 	)
 	(segment
-		(start 112.765 115.975)
-		(end 121.59 124.8)
-		(width 0.15)
-		(layer "F.Cu")
-		(net 34)
-	)
-	(segment
 		(start 109.375 115.975)
 		(end 109.375 111.85)
@@
 	)
 	(segment
-		(start 109.375 115.975)
-		(end 112.765 115.975)
-		(width 0.15)
-		(layer "F.Cu")
-		(net 34)
-	)
-	(segment
 		(start 101.8 104.8965)
 		(end 101.8 106)
@@
 		(polygon
 			(pts
-				(xy 142.25 108.5) (xy 149.25 108.5) (xy 149.25 115.25) (xy 142.25 115.25)
+				(xy 142.25 108.5) (xy 149.25 108.5) (xy 149.25 115.35) (xy 142.25 115.35)
 			)
 		)
@@
 		(polygon
 			(pts
-				(xy 145.3 103.7) (xy 145.3 108.1) (xy 141.8 108.1) (xy 141.8 105) (xy 143.1 103.7)
+				(xy 145.3 103.7) (xy 145.3 108.5) (xy 141.8 108.5) (xy 141.8 105) (xy 143.1 103.7)
 			)
 		)
