File: RP-006442-DD-2-RP2350B Minimal Board Kicad archive/buttons.kicad_sch (KiCad schematic)
At the start: 5 parts, among them SW10 SW_DIP_x08, SW5 SW_Push, SW6 SW_Push, SW7 SW_Push, SW8 SW_Push

Commit message: Created Figures
Other:
- moved on the sheet: SW10, SW5, SW6, SW7, SW8
